Commit message: updated torso to have new links

File: nefive_description/urdf/torso.xacro (robot description, xacro)
@@ -28,4 +28,5 @@
     </visual>
   </link>
+  <link name="shoulder_centre" />
   <joint name="base_link_lower_torso_joint" type="fixed">
     <origin rpy="0 5.497787 0" xyz="-0.0241 0 0.0285" />
@@ -46,5 +47,10 @@
     <origin xyz="0.025 0 0.075" />
     <parent link="chest_box" />
-    <child link="arms" />
+    <child link="shoulder_centre" />
+  </joint>
+  <joint name="shoulder_centre_left_arm_joint" type="fixed">
+    <origin xyz="-0.10 0 0" />
+    <parent link="shoulder_centre" />
+    <child link="left_arm" />
   </joint>
 </robot>
