Commit message: switched to a multicamera, tweaked the links rpy

File: nefive_description/urdf/nefive.urdf (robot description, URDF)
Before this commit: robot nefive, 43 links, 42 joints
Links:
- removed link left_camera
- added link left_camera_pointcloud_frame, mass 0.001
Joints:
- joint left_eye_inner_left_camera_joint: child left_camera -> left_camera_pointcloud_frame; origin (none) -> xyz=0 0 0 rpy=-1.57 0 -1.57 

Commit message: fixed the issue with skid steer I had the collider on the right front wheel interecting with the body of the robot!

File: nefive_description/urdf/nefive.urdf (robot description, URDF)
Before this commit: robot nefive, 43 links, 42 joints
Joints:
- joint left_eye_inner_left_camera_joint: origin xyz=0 0 0 rpy=-1.57 0 -1.57  -> rpy=-1.57 0 -1.57
- joint right_forearm_right_wrist_roll_joint: origin xyz=0.0683 -0.0025 0 rpy=0 4.712389 0 -> xyz=0.0683 -0.0025 0 rpy=0 4.712734 0

Commit message: updated urdf, generated from the xacro

File: nefive_description/urdf/nefive.urdf (robot description, URDF)
Before this commit: robot nefive, 43 links, 42 joints
Links:
- removed link left_forearm
- removed link left_shoulder_pan
- removed link left_shoulder_tilt
- removed link left_wrist_roll
- removed link rear_left_idler
- removed link rear_right_idler
- removed link right_forearm
- removed link right_shoulder_pan
- removed link right_shoulder_tilt
- removed link right_wrist_roll
- removed link upper_tracks
- added link left_shoulder_flappy; visual cylinder length=0.02 radius=0.0005
- added link left_shoulder_foreaft; visual cylinder length=0.004 radius=0.0005
- added link left_wrist_rotate; visual cylinder length=0.004 radius=0.0005; visual cylinder length=0.034 radius=0.005
- added link right_shoulder_flappy; visual cylinder length=0.02 radius=0.0005
- added link right_shoulder_foreaft; visual cylinder length=0.004 radius=0.0005
- added link right_wrist_rotate; visual cylinder length=0.004 radius=0.0005; visual cylinder length=0.034 radius=0.005
- added link shoulder_centre
- link arms: mass 0.001 -> None
- link chassis: mass 0.001 -> None; geometry visual box size=0.104 0.147 0.068
- link chest_box: mass 0.001 -> None; geometry visual box size=0.05 0.07 0.05
- link eyes: mass 0.001 -> None; geometry visual cylinder length=0 radius=0
- link front_left_wheel: mass 0.001 -> None; geometry visual cylinder length=0.02 radius=0.025
- link front_right_wheel: mass 0.001 -> None; geometry visual cylinder length=0.02 radius=0.025
- link head: mass 0.001 -> None; geometry visual box size=0.107 0.11 0.054
- link head_pan: mass 0.001 -> None; geometry visual cylinder length=0.002 radius=0.02
- link head_tilt: mass 0.001 -> None; geometry visual box size=0.04 0.04 0.001
- link left_arm: mass 0.001 -> None
- link left_camera_pointcloud_frame: mass 0.001 -> None
- link left_elbow: mass 0.001 -> None; geometry visual cylinder length=0.004 radius=0.0005; visual cylinder length=0.042 radius=0.005
- link left_eye_inner: mass 0.001 -> None; geometry visual cylinder length=0.002 radius=0.01
- link left_eye_ring: mass 0.001 -> None; geometry visual cylinder length=0.002 radius=0.02
- link left_hand: mass 0.001 -> None
- link left_shoulder_rotate: mass 0.001 -> None; geometry visual cylinder length=0.004 radius=0.0005; visual cylinder length=0.06 radius=0.005
- link left_wrist_pan: mass 0.001 -> None; geometry visual cylinder length=0.01 radius=0.0005; visual cylinder length=0.032 radius=0.005
- link left_wrist_tilt: mass 0.001 -> None; geometry visual cylinder length=0.01 radius=0.0005
- link lower_torso: mass 0.001 -> None; geometry visual box size=0.015 0.06 0.06
- link rear_left_wheel: mass 0.001 -> None; geometry visual cylinder length=0.02 radius=0.025
- link rear_right_wheel: mass 0.001 -> None; geometry visual cylinder length=0.02 radius=0.025
- link right_arm: mass 0.001 -> None
- link right_camera: mass 0.001 -> None
- link right_elbow: mass 0.001 -> None; geometry visual cylinder length=0.004 radius=0.0005; visual cylinder length=0.042 radius=0.005
- link right_eye_inner: mass 0.001 -> None; geometry visual cylinder length=0.002 radius=0.01
- link right_eye_ring: mass 0.001 -> None; geometry visual cylinder length=0.002 radius=0.02
- link right_hand: mass 0.001 -> None
- link right_shoulder_rotate: mass 0.001 -> None; geometry visual cylinder length=0.004 radius=0.0005; visual cylinder length=0.06 radius=0.005
- link right_wrist_pan: mass 0.001 -> None; geometry visual cylinder length=0.01 radius=0.0005; visual cylinder length=0.032 radius=0.005
- link right_wrist_tilt: mass 0.001 -> None; geometry visual cylinder length=0.01 radius=0.0005
- link upper_torso: mass 0.001 -> None; geometry visual box size=0.015 0.06 0.06
Joints:
- removed joint 
- removed joint arms_left_arm_joint
- removed joint arms_right_arm_joint
- removed joint base_link_rear_left_idler_joint
- removed joint base_link_rear_right_idler_joint
- removed joint left_arm_left_shoulder_tilt_joint
- removed joint left_elbow_left_forearm_joint
- removed joint left_forearm_left_wrist_roll_joint
- removed joint left_shoulder_pan_left_shoulder_rotate_joint
- removed joint left_shoulder_tilt_left_shoulder_pan_joint
- removed joint left_wrist_pan_left_hand_joint
- removed joint left_wrist_roll_left_wrist_tilt_joint
- removed joint left_wrist_tilt_left_wrist_pan_joint
- removed joint right_arm_right_shoulder_tilt_joint
- removed joint right_elbow_right_forearm_joint
- removed joint right_forearm_right_wrist_roll_joint
- removed joint right_shoulder_pan_right_shoulder_rotate_joint
- removed joint right_shoulder_tilt_right_shoulder_pan_joint
- removed joint right_wrist_pan_right_hand_joint
- removed joint right_wrist_roll_right_wrist_tilt_joint
- removed joint right_wrist_tilt_right_wrist_pan_joint
- added joint arms_left_arm: type fixed, parent arms, child left_arm, origin xyz=-0.075 0 0 rpy=0 0 0
- added joint arms_right_arm: type fixed, parent arms, child right_arm, origin xyz=0.075 0 0 rpy=0 0 0
- added joint left_arm_left_shoulder_flappy_joint: type revolute, parent left_arm, child left_shoulder_flappy, origin xyz=0 0 0 rpy=0 0 0, axis 0 -1 0, limit lower=-1.5707963267948966 upper=1.5707963267948966 effort=10 velocity=1000
- added joint left_forearm_left_wrist_rotate_joint: type revolute, parent left_elbow, child left_wrist_rotate, origin xyz=0.042 0 0 rpy=0 0 0, axis 1 0 0, limit lower=-1.5707963267948966 upper=1.5707963267948966 effort=10 velocity=1000
- added joint left_shoulder_flappy_left_shoulder_foreaft_joint: type revolute, parent left_shoulder_flappy, child left_shoulder_foreaft, origin xyz=-0.025 0 0 rpy=0 0 0, axis 1 0 0, limit lower=-1.5707963267948966 upper=1.5707963267948966 effort=10 velocity=1000
- added joint left_shoulder_foreaft_left_shoulder_rotate_joint: type revolute, parent left_shoulder_foreaft, child left_shoulder_rotate, origin xyz=0 0 -0.067 rpy=0 0 -1.5707963267948966, axis 0 0 -1, limit lower=-1.5707963267948966 upper=1.5707963267948966 effort=10 velocity=1000
- added joint left_wrist_pan_left_wrist_tilt_joint: type revolute, parent left_wrist_pan, child left_wrist_tilt, origin xyz=0.036 0 0 rpy=1.57 0 0, axis 0 0 1, limit lower=-1.5707963267948966 upper=1.5707963267948966 effort=10 velocity=1000
- added joint left_wrist_rotate_left_wrist_pan_joint: type revolute, parent left_wrist_rotate, child left_wrist_pan, origin xyz=0.034 0 0 rpy=0 0 0, axis 0 0 1, limit lower=-1.5707963267948966 upper=1.5707963267948966 effort=10 velocity=1000
- added joint left_wrist_tilt_left_hand_joint: type fixed, parent left_wrist_tilt, child left_hand, origin xyz=0.012 0 0
- added joint right_arm_right_shoulder_flappy_joint: type revolute, parent right_arm, child right_shoulder_flappy, origin xyz=0 0 0 rpy=0 0 0, axis 0 -1 0, limit lower=-1.5707963267948966 upper=1.5707963267948966 effort=10 velocity=1000
- added joint right_forearm_right_wrist_rotate_joint: type revolute, parent right_elbow, child right_wrist_rotate, origin xyz=0.042 0 0 rpy=0 0 0, axis 1 0 0, limit lower=-1.5707963267948966 upper=1.5707963267948966 effort=10 velocity=1000
- added joint right_shoulder_flappy_right_shoulder_foreaft_joint: type revolute, parent right_shoulder_flappy, child right_shoulder_foreaft, origin xyz=0.025 0 0 rpy=0 0 0, axis -1 0 0, limit lower=-1.5707963267948966 upper=1.5707963267948966 effort=10 velocity=1000
- added joint right_shoulder_foreaft_right_shoulder_rotate_joint: type revolute, parent right_shoulder_foreaft, child right_shoulder_rotate, origin xyz=0 0 -0.067 rpy=0 0 -1.5707963267948966, axis 0 0 -1, limit lower=-1.5707963267948966 upper=1.5707963267948966 effort=10 velocity=1000
- added joint right_wrist_pan_right_wrist_tilt_joint: type revolute, parent right_wrist_pan, child right_wrist_tilt, origin xyz=0.036 0 0 rpy=1.57 0 0, axis 0 0 -1, limit lower=-1.5707963267948966 upper=1.5707963267948966 effort=10 velocity=1000
- added joint right_wrist_rotate_right_wrist_pan_joint: type revolute, parent right_wrist_rotate, child right_wrist_pan, origin xyz=0.034 0 0 rpy=0 0 0, axis 0 0 1, limit lower=-1.5707963267948966 upper=1.5707963267948966 effort=10 velocity=1000
- added joint right_wrist_tilt_right_hand_joint: type fixed, parent right_wrist_tilt, child right_hand, origin xyz=0.012 0 0
- added joint shoulder_centre_arms_joint: type fixed, parent shoulder_centre, child arms, origin xyz=0 0 0 rpy=0 0 0
- joint chest_box_arms_joint: child arms -> shoulder_centre; origin xyz=0.025 0 0.075 -> xyz=0.025 0 0.075 rpy=0 0 -1.570451
- joint left_shoulder_rotate_left_elbow_joint: axis 0 -1 0 -> 0 1 0; limit lower=0 upper=0 effort=1000 velocity=1000 -> lower=-1.5707963267948966 upper=1.5707963267948966 effort=10 velocity=1000; origin xyz=0.075 0 0 -> xyz=0 0 0 rpy=0 3.141592653589793 0
- joint right_shoulder_rotate_right_elbow_joint: limit lower=0 upper=0 effort=1000 velocity=1000 -> lower=-1.5707963267948966 upper=1.5707963267948966 effort=10 velocity=1000; origin xyz=0.075 0 0 -> xyz=0 0 0 rpy=0 3.141592653589793 0
