Commit message: added rviz bits, arms_only urdf

File: nefive_description/urdf/arms.xacro (robot description, xacro)
@@ -175,9 +175,4 @@
     </visual>
   </link>
-<joint name="chest_box_arms_joint" type="fixed">
-    <origin xyz="0.025 0 0.075" />
-    <parent link="chest_box" />
-    <child link="arms" />
-  </joint>
   <joint name="arms_right_arm_joint" type="fixed">
     <origin xyz="0 -0.06 0" />

File: nefive_description/urdf/nefive-simplified.urdf.xacro (robot description, xacro)
@@ -1,13 +1,5 @@
 ﻿<?xml version="1.0" encoding="utf-8"?>
 <robot xmlns:xacro="http://www.ros.org/wiki/xacro" name="nefive">
-  <material name="grey">
-    <color rgba="0.5 0.5 0.5 1" />
-  </material>
-  <material name="black">
-    <color rgba="0 0 0 1" />
-  </material>
-  <material name="Default-Material">
-    <color rgba="1 1 1 1" />
-  </material>
+  <xacro:include filename="materials.xacro" />
   <xacro:include filename="base.xacro" />
   <xacro:include filename="wheels.xacro" />

File: nefive_description/urdf/torso.xacro (robot description, xacro)
@@ -43,3 +43,8 @@
     <child link="chest_box" />
   </joint>
+  <joint name="chest_box_arms_joint" type="fixed">
+    <origin xyz="0.025 0 0.075" />
+    <parent link="chest_box" />
+    <child link="arms" />
+  </joint>
 </robot>

Commit message: currently actually rendering...

File: nefive_description/urdf/arms.xacro (robot description, xacro)
@@ -1,97 +1,8 @@
 <?xml version="1.0"?>
-<robot xmlns:xacro="http://www.ros.org/wiki/xacro" >
-<link name="arms">
-  </link>
-  <link name="right_arm">
-  </link>
-    <link name="right_shoulder_tilt">
-      <visual>
-        <origin rpy="0 1.570451 0" />
-        <geometry>
-          <cylinder length="0.02" radius="0.0005" />
-        </geometry>
-        <material name="grey" />
-      </visual>
-    </link>
-    <link name="right_shoulder_pan">
-      <visual>
-        <origin rpy="-4.712389 0 0" xyz="0 -0.002 0" />
-        <geometry>
-          <cylinder length="0.004" radius="0.0005" />
-        </geometry>
-        <material name="grey" />
-      </visual>
-    </link>
-    <link name="right_shoulder_rotate">
-      <visual>
-        <origin rpy="-4.712389 0 -4.712389" xyz="0.0001 -0.002 0" />
-        <geometry>
-          <cylinder length="0.004" radius="0.0005" />
-        </geometry>
-        <material name="grey" />
-      </visual>
-      <visual>
-        <origin rpy="0 1.570451 0" xyz="0.031 -0.002 0" />
-        <geometry>
-          <cylinder length="-0.06" radius="0.005" />
-        </geometry>
-        <material name="grey" />
-      </visual>
-    </link>
-    <link name="right_elbow">
-      <visual>
-        <origin rpy="0 1.570451 0" />
-        <geometry>
-          <cylinder length="0.02" radius="0.0005" />
-        </geometry>
-        <material name="grey" />
-      </visual>
-    </link>
-    <link name="right_forearm">
-      <visual>
-        <origin rpy="0 1.570451 0" xyz="0.035 -0.0025 0" />
-        <geometry>
-          <cylinder length="0.07" radius="0.005" />
-        </geometry>
-        <material name="grey" />
-      </visual>
-    </link>
-    <link name="right_wrist_roll">
-      <visual>
-        <geometry>
-          <cylinder length="0.01" radius="0.0005" />
-        </geometry>
-        <material name="grey" />
-      </visual>
-    </link>
-    <link name="right_wrist_tilt">
-      <visual>
-        <geometry>
-          <cylinder length="0.01" radius="0.0005" />
-        </geometry>
-        <material name="grey" />
-      </visual>
-    </link>
-    <link name="right_wrist_pan">
-      <visual>
-        <geometry>
-          <cylinder length="0.01" radius="0.0005" />
-        </geometry>
-        <material name="grey" />
-      </visual>
-    </link>
-    <link name="right_hand">
-      <visual>
-        <geometry>
-          <box size="0.02 0.02 0.02" />
-        </geometry>
-        <material name="grey" />
-      </visual>
-    </link>
-  <link name="left_arm">
-  </link>
-  <link name="left_shoulder_tilt">
+<robot xmlns:xacro="http://www.ros.org/wiki/xacro">
+  <link name="left_arm" />
+  <link name="left_shoulder_flappy">
     <visual>
-      <origin rpy="0 1.570451 0" />
+      <origin rpy="1.570451 0 0" xyz="0 0 0" />
       <geometry>
         <cylinder length="0.02" radius="0.0005" />
@@ -100,7 +11,7 @@
     </visual>
   </link>
-  <link name="left_shoulder_pan">
+  <link name="left_shoulder_foreaft">
     <visual>
-      <origin rpy="-4.712389 0 0" xyz="0 -0.002 0" />
+      <origin rpy="0 0 0" xyz="0 -0.002 0" />
       <geometry>
         <cylinder length="0.004" radius="0.0005" />
@@ -151,5 +62,5 @@
     </visual>
   </link>
-  <link name="left_wrist_tilt">
+  <link name="left_wrist_flappy">
     <visual>
       <geometry>
@@ -175,95 +86,24 @@
     </visual>
   </link>
-  <joint name="arms_right_arm_joint" type="fixed">
-    <origin xyz="0 -0.06 0" />
-    <parent link="arms" />
-    <child link="right_arm" />
+  <joint name="left_arm_left_shoulder_flappy_joint" type="revolute">
+    <origin rpy="0 0 0" xyz="0 0 0" />
+    <parent link="left_arm" />
+    <child link="left_shoulder_flappy" />
+    <axis xyz="0 1 0" />
+    <limit effort="1000" lower="-1.570796" upper="1.570796" velocity="1000" />
   </joint>
-  <joint name="right_arm_right_shoulder_tilt_joint" type="revolute">
-    <origin rpy="0 0.785398 0" />
-    <parent link="right_arm" />
-    <child link="right_shoulder_tilt" />
+  <joint name="left_shoulder_flappy_left_shoulder_foreaft_joint" type="revolute">
+    <origin rpy="0 0 0" xyz="-0.025 0 0" />
+    <parent link="left_shoulder_flappy" />
+    <child link="left_shoulder_foreaft" />
     <axis xyz="1 0 0" />
-    <limit lower="-0.610865" upper="0.436332" effort="1000" velocity="1000" />
+    <limit effort="1000" lower="-1.570796" upper="1.570796" velocity="1000" />
   </joint>
-  <joint name="right_shoulder_tilt_right_shoulder_pan_joint" type="revolute">
-    <origin rpy="0 0.785398 0" xyz="0 -0.001 0" />
-    <parent link="right_shoulder_tilt" />
-    <child link="right_shoulder_pan" />
-    <axis xyz="0 -1 0" />
-    <limit lower="-1.570796" upper="1.570796" effort="1000" velocity="1000" />
-  </joint>
-  <joint name="right_shoulder_pan_right_shoulder_rotate_joint" type="revolute">
-    <origin rpy="0 0.785398 0" xyz="0 -0.0048 0" />
-    <parent link="right_shoulder_pan" />
-    <child link="right_shoulder_rotate" />
-    <axis xyz="1 0 0" />
-    <limit lower="-1.570796" upper="1.570796" effort="1000" velocity="1000" />
-  </joint>
-  <joint name="right_shoulder_rotate_right_elbow_joint" type="revolute">
-    <origin xyz="0.075 0 0" />
-    <parent link="right_shoulder_rotate" />
-    <child link="right_elbow" />
-    <axis xyz="0 -1 0" />
-    <limit lower="0" upper="0" effort="1000" velocity="1000" />
-  </joint>
-  <joint name="right_elbow_right_forearm_joint" type="revolute">
-    <origin rpy="-3.141593 5.497787 -3.141593" xyz="0.01 0 0.0025" />
-    <parent link="right_elbow" />
-    <child link="right_forearm" />
-    <axis xyz="0 -1 0" />
-    <limit lower="0" upper="0" effort="1000" velocity="1000" />
-  </joint>
-  <joint name="right_forearm_right_wrist_roll_joint" type="revolute">
-    <origin rpy="0 4.712734 0" xyz="0.0683 -0.0025 0" />
-    <parent link="right_forearm" />
-    <child link="right_wrist_roll" />
+  <joint name="left_shoulder_foreaft_left_shoulder_rotate_joint" type="revolute">
+    <origin rpy="0 0 0" xyz="0 0 -0.067" />
+    <parent link="left_shoulder_foreaft" />
+    <child link="left_shoulder_rotate" />
     <axis xyz="0 0 1" />
-    <limit lower="-1.570796" upper="1.570796" effort="1000" velocity="1000" />
-  </joint>
-  <joint name="right_wrist_roll_right_wrist_tilt_joint" type="revolute">
-    <origin rpy="0 1.570796 -4.712389" xyz="0 0 -0.00636" />
-    <parent link="right_wrist_roll" />
-    <child link="right_wrist_tilt" />
-    <axis xyz="0 0 1" />
-    <limit lower="-0.785398" upper="0.785398" effort="1000" velocity="1000" />
-  </joint>
-  <joint name="right_wrist_tilt_right_wrist_pan_joint" type="revolute">
-    <origin rpy="-4.712389 0 0" xyz="0.002 0 0" />
-    <parent link="right_wrist_tilt" />
-    <child link="right_wrist_pan" />
-    <axis xyz="0 0 1" />
-    <limit lower="-0.785398" upper="0.785398" effort="1000" velocity="1000" />
-  </joint>
-  <joint name="right_wrist_pan_right_hand_joint" type="fixed">
-    <origin xyz="0.012 0 0" />
-    <parent link="right_wrist_pan" />
-    <child link="right_hand" />
-  </joint>
-  <joint name="arms_left_arm_joint" type="fixed">
-    <origin rpy="0 0 -3.141593" xyz="0 0.06 0" />
-    <parent link="arms" />
-    <child link="left_arm" />
-  </joint>
-  <joint name="left_arm_left_shoulder_tilt_joint" type="revolute">
-    <origin rpy="0 5.497787 0" />
-    <parent link="left_arm" />
-    <child link="left_shoulder_tilt" />
-    <axis xyz="1 0 0" />
-    <limit lower="-0.610865" upper="0.436332" effort="1000" velocity="1000" />
-  </joint>
-  <joint name="left_shoulder_tilt_left_shoulder_pan_joint" type="revolute">
-    <origin rpy="-3.141593 0.785398 -3.141593" xyz="0 -0.001 0" />
-    <parent link="left_shoulder_tilt" />
-    <child link="left_shoulder_pan" />
-    <axis xyz="0 -1 0" />
-    <limit lower="-1.570796" upper="1.570796" effort="1000" velocity="1000" />
-  </joint>
-  <joint name="left_shoulder_pan_left_shoulder_rotate_joint" type="revolute">
-    <origin rpy="0 5.497787 0" xyz="0 -0.0048 0" />
-    <parent link="left_shoulder_pan" />
-    <child link="left_shoulder_rotate" />
-    <axis xyz="1 0 0" />
-    <limit lower="-1.570796" upper="1.570796" effort="1000" velocity="1000" />
+    <limit effort="1000" lower="-1.570796" upper="1.570796" velocity="1000" />
   </joint>
   <joint name="left_shoulder_rotate_left_elbow_joint" type="revolute">
@@ -272,5 +112,5 @@
     <child link="left_elbow" />
     <axis xyz="0 -1 0" />
-    <limit lower="0" upper="0" effort="1000" velocity="1000" />
+    <limit effort="1000" lower="0" upper="0" velocity="1000" />
   </joint>
   <joint name="left_elbow_left_forearm_joint" type="revolute">
@@ -279,5 +119,5 @@
     <child link="left_forearm" />
     <axis xyz="0 -1 0" />
-    <limit lower="0" upper="0" effort="1000" velocity="1000" />
+    <limit effort="1000" lower="0" upper="0" velocity="1000" />
   </joint>
   <joint name="left_forearm_left_wrist_roll_joint" type="revolute">
@@ -286,19 +126,19 @@
     <child link="left_wrist_roll" />
     <axis xyz="0 0 1" />
-    <limit lower="-1.570796" upper="1.570796" effort="1000" velocity="1000" />
+    <limit effort="1000" lower="-1.570796" upper="1.570796" velocity="1000" />
   </joint>
-  <joint name="left_wrist_roll_left_wrist_tilt_joint" type="revolute">
+  <joint name="left_wrist_roll_left_wrist_flappy_joint" type="revolute">
     <origin rpy="0 1.570796 -4.712389" xyz="0 0 -0.00636" />
     <parent link="left_wrist_roll" />
-    <child link="left_wrist_tilt" />
+    <child link="left_wrist_flappy" />
     <axis xyz="0 0 1" />
-    <limit lower="-0.785398" upper="0.785398" effort="1000" velocity="1000" />
+    <limit effort="1000" lower="-0.785398" upper="0.785398" velocity="1000" />
   </joint>
-  <joint name="left_wrist_tilt_left_wrist_pan_joint" type="revolute">
+  <joint name="left_wrist_flappy_left_wrist_pan_joint" type="revolute">
     <origin rpy="-4.712389 0 0" xyz="0.002 0 0" />
-    <parent link="left_wrist_tilt" />
+    <parent link="left_wrist_flappy" />
     <child link="left_wrist_pan" />
     <axis xyz="0 0 1" />
-    <limit lower="-0.785398" upper="0.785398" effort="1000" velocity="1000" />
+    <limit effort="1000" lower="-0.785398" upper="0.785398" velocity="1000" />
   </joint>
   <joint name="left_wrist_pan_left_hand_joint" type="fixed">
@@ -307,3 +147,3 @@
     <child link="left_hand" />
   </joint>
-</robot>
+  </robot>

File: nefive_description/urdf/just_arms.urdf.xacro (robot description, xacro)
@@ -2,8 +2,38 @@
 <robot name="ne-five-arms" xmlns:xacro="http://www.ros.org/wiki/xacro" >
   <link name="base_link" />
-  <joint name="base_link_arms_joint" type="fixed">
+  <link name="shoulder_centre" />
+  <joint name="shoulder_centre_left_arm_joint" type="fixed">
+    <origin xyz="-0.10 0 0" />
+    <parent link="shoulder_centre" />
+    <child link="left_arm" />
+  </joint>
+  <link name="forward_indicator" />
+  <link name="backward_indicator" />
+  <link name="left_indicator" />
+  <link name="right_indicator" />
+  <joint name="base_link_forward_indicator" type="fixed">
+    <origin xyz="0 0.1 0" />
+    <parent link="base_link" />
+    <child link="forward_indicator" />
+  </joint>
+  <joint name="base_link_backward_indicator" type="fixed">
+    <origin xyz="0 -0.1 0" />
+    <parent link="base_link" />
+    <child link="backward_indicator" />
+  </joint>
+  <joint name="base_link_left_indicator" type="fixed">
+    <origin xyz="-0.1 0 0" />
+    <parent link="base_link" />
+    <child link="left_indicator" />
+  </joint>
+  <joint name="base_link_right_indicator" type="fixed">
+    <origin xyz="0.1 0 0" />
+    <parent link="base_link" />
+    <child link="right_indicator" />
+  </joint>
+  <joint name="base_link_shoulder_centre" type="fixed">
     <origin xyz="0 0 0.24" />
     <parent link="base_link" />
-    <child link="arms" />
+    <child link="shoulder_centre" />
   </joint>
   <xacro:include filename="arms.xacro" />

File: nefive_description/urdf/materials.xacro (robot description, xacro)
@@ -1,6 +1,9 @@
 <?xml version="1.0"?>
 <robot xmlns:xacro="http://www.ros.org/wiki/xacro" >
-    <material name="grey">
+  <material name="grey">
     <color rgba="0.5 0.5 0.5 1" />
+  </material>
+  <material name="green">
+    <color rgba="0 0.5 0 1" />
   </material>
   <material name="black">

Commit message: rotating around shoulder_foreaft

File: nefive_description/urdf/arms.xacro (robot description, xacro)
@@ -13,14 +13,14 @@
   <link name="left_shoulder_foreaft">
     <visual>
-      <origin rpy="0 0 0" xyz="0 -0.002 0" />
+      <origin rpy="0 1.570451 0" xyz="0 0 0" />
       <geometry>
         <cylinder length="0.004" radius="0.0005" />
       </geometry>
-      <material name="grey" />
+      <material name="green" />
     </visual>
   </link>
   <link name="left_shoulder_rotate">
     <visual>
-      <origin rpy="-4.712389 0 -4.712389" xyz="0.0001 -0.002 0" />
+      <origin rpy="-4.712389 0 -4.712389" xyz="0 0 0" />
       <geometry>
         <cylinder length="0.004" radius="0.0005" />

Commit message: upper_arm cylinder in position

File: nefive_description/urdf/arms.xacro (robot description, xacro)
@@ -17,10 +17,10 @@
         <cylinder length="0.004" radius="0.0005" />
       </geometry>
-      <material name="green" />
+      <material name="grey" />
     </visual>
   </link>
   <link name="left_shoulder_rotate">
     <visual>
-      <origin rpy="-4.712389 0 -4.712389" xyz="0 0 0" />
+      <origin rpy="0 0 0" xyz="0 0 0" />
       <geometry>
         <cylinder length="0.004" radius="0.0005" />
@@ -29,9 +29,9 @@
     </visual>
     <visual>
-      <origin rpy="0 1.570451 0" xyz="0.031 -0.002 0" />
+      <origin rpy="0 0 0" xyz="0 0 0.03" />
       <geometry>
-        <cylinder length="-0.06" radius="0.005" />
+        <cylinder length="0.06" radius="0.005" />
       </geometry>
-      <material name="grey" />
+      <material name="green" />
     </visual>
   </link>

Commit message: elbow working

File: nefive_description/urdf/arms.xacro (robot description, xacro)
@@ -33,12 +33,12 @@
         <cylinder length="0.06" radius="0.005" />
       </geometry>
-      <material name="green" />
+      <material name="grey" />
     </visual>
   </link>
   <link name="left_elbow">
     <visual>
-      <origin rpy="0 1.570451 0" />
+      <origin rpy="1.570451 0 0" xyz="0 0 0" />
       <geometry>
-        <cylinder length="0.02" radius="0.0005" />
+        <cylinder length="0.004" radius="0.0005" />
       </geometry>
       <material name="grey" />
@@ -47,5 +47,5 @@
   <link name="left_forearm">
     <visual>
-      <origin rpy="0 1.570451 0" xyz="0.035 -0.0025 0" />
+      <origin rpy="0 1.570451 0" xyz="0.035 0 0" />
       <geometry>
         <cylinder length="0.07" radius="0.005" />
@@ -101,5 +101,5 @@
   </joint>
   <joint name="left_shoulder_foreaft_left_shoulder_rotate_joint" type="revolute">
-    <origin rpy="0 0 0" xyz="0 0 -0.067" />
+    <origin rpy="0 0 -1.570451" xyz="0 0 -0.067" />
     <parent link="left_shoulder_foreaft" />
     <child link="left_shoulder_rotate" />
@@ -108,16 +108,16 @@
   </joint>
   <joint name="left_shoulder_rotate_left_elbow_joint" type="revolute">
-    <origin xyz="0.075 0 0" />
+    <origin rpy="0 0 0" xyz="0 0 0" />
     <parent link="left_shoulder_rotate" />
     <child link="left_elbow" />
     <axis xyz="0 -1 0" />
-    <limit effort="1000" lower="0" upper="0" velocity="1000" />
+    <limit effort="1000" lower="-1" upper="1" velocity="1000" />
   </joint>
   <joint name="left_elbow_left_forearm_joint" type="revolute">
-    <origin rpy="-3.141593 0.785398 -3.141593" xyz="0.01 0 0.0025" />
+    <origin rpy="-3.141593 0.785398 -3.141593" xyz="0 0 0" />
     <parent link="left_elbow" />
     <child link="left_forearm" />
     <axis xyz="0 -1 0" />
-    <limit effort="1000" lower="0" upper="0" velocity="1000" />
+    <limit effort="1000" lower="-1" upper="1" velocity="1000" />
   </joint>
   <joint name="left_forearm_left_wrist_roll_joint" type="revolute">

Commit message: elbow working, oriented correctly

File: nefive_description/urdf/arms.xacro (robot description, xacro)
@@ -44,6 +44,4 @@
       <material name="grey" />
     </visual>
-  </link>
-  <link name="left_forearm">
     <visual>
       <origin rpy="0 1.570451 0" xyz="0.035 0 0" />
@@ -108,20 +106,13 @@
   </joint>
   <joint name="left_shoulder_rotate_left_elbow_joint" type="revolute">
-    <origin rpy="0 0 0" xyz="0 0 0" />
+    <origin rpy="0 3.14 0" xyz="0 0 0" />
     <parent link="left_shoulder_rotate" />
     <child link="left_elbow" />
-    <axis xyz="0 -1 0" />
-    <limit effort="1000" lower="-1" upper="1" velocity="1000" />
-  </joint>
-  <joint name="left_elbow_left_forearm_joint" type="revolute">
-    <origin rpy="-3.141593 0.785398 -3.141593" xyz="0 0 0" />
-    <parent link="left_elbow" />
-    <child link="left_forearm" />
-    <axis xyz="0 -1 0" />
+    <axis xyz="0 1 0" />
     <limit effort="1000" lower="-1" upper="1" velocity="1000" />
   </joint>
   <joint name="left_forearm_left_wrist_roll_joint" type="revolute">
     <origin rpy="0 4.712734 0" xyz="0.0683 -0.0025 0" />
-    <parent link="left_forearm" />
+    <parent link="left_elbow" />
     <child link="left_wrist_roll" />
     <axis xyz="0 0 1" />

Commit message: wrist rotate, done

File: nefive_description/urdf/arms.xacro (robot description, xacro)
@@ -45,15 +45,16 @@
     </visual>
     <visual>
-      <origin rpy="0 1.570451 0" xyz="0.035 0 0" />
+      <origin rpy="0 1.570451 0" xyz="0.021 0 0" />
       <geometry>
-        <cylinder length="0.07" radius="0.005" />
+        <cylinder length="0.042" radius="0.005" />
       </geometry>
       <material name="grey" />
     </visual>
   </link>
-  <link name="left_wrist_roll">
+  <link name="left_wrist_rotate">
     <visual>
+      <origin rpy="0 1.570451 0" xyz="0 0 0" />
       <geometry>
-        <cylinder length="0.01" radius="0.0005" />
+        <cylinder length="0.004" radius="0.0005" />
       </geometry>
       <material name="grey" />
@@ -112,14 +113,14 @@
     <limit effort="1000" lower="-1" upper="1" velocity="1000" />
   </joint>
-  <joint name="left_forearm_left_wrist_roll_joint" type="revolute">
-    <origin rpy="0 4.712734 0" xyz="0.0683 -0.0025 0" />
+  <joint name="left_forearm_left_wrist_rotate_joint" type="revolute">
+    <origin rpy="0 0 0" xyz="0.042 0 0" />
     <parent link="left_elbow" />
-    <child link="left_wrist_roll" />
-    <axis xyz="0 0 1" />
+    <child link="left_wrist_rotate" />
+    <axis xyz="1 0 0" />
     <limit effort="1000" lower="-1.570796" upper="1.570796" velocity="1000" />
   </joint>
-  <joint name="left_wrist_roll_left_wrist_flappy_joint" type="revolute">
+  <joint name="left_wrist_rotate_left_wrist_flappy_joint" type="revolute">
     <origin rpy="0 1.570796 -4.712389" xyz="0 0 -0.00636" />
-    <parent link="left_wrist_roll" />
+    <parent link="left_wrist_rotate" />
     <child link="left_wrist_flappy" />
     <axis xyz="0 0 1" />

Commit message: wrist rotate visual added

File: nefive_description/urdf/arms.xacro (robot description, xacro)
@@ -60,6 +60,13 @@
       <material name="grey" />
     </visual>
+    <visual>
+      <origin rpy="0 1.570451 0" xyz="0.017 0 0" />
+      <geometry>
+        <cylinder length="0.034" radius="0.005" />
+      </geometry>
+      <material name="green" />
+    </visual>
   </link>
-  <link name="left_wrist_flappy">
+  <link name="left_wrist_pan">
     <visual>
       <geometry>
@@ -69,5 +76,5 @@
     </visual>
   </link>
-  <link name="left_wrist_pan">
+  <link name="left_wrist_pan_old">
     <visual>
       <geometry>
@@ -120,21 +127,21 @@
     <limit effort="1000" lower="-1.570796" upper="1.570796" velocity="1000" />
   </joint>
-  <joint name="left_wrist_rotate_left_wrist_flappy_joint" type="revolute">
-    <origin rpy="0 1.570796 -4.712389" xyz="0 0 -0.00636" />
+  <joint name="left_wrist_rotate_left_wrist_pan_joint" type="revolute">
+    <origin rpy="0 0 0" xyz="0.034 0 0" />
     <parent link="left_wrist_rotate" />
-    <child link="left_wrist_flappy" />
-    <axis xyz="0 0 1" />
-    <limit effort="1000" lower="-0.785398" upper="0.785398" velocity="1000" />
-  </joint>
-  <joint name="left_wrist_flappy_left_wrist_pan_joint" type="revolute">
-    <origin rpy="-4.712389 0 0" xyz="0.002 0 0" />
-    <parent link="left_wrist_flappy" />
     <child link="left_wrist_pan" />
     <axis xyz="0 0 1" />
     <limit effort="1000" lower="-0.785398" upper="0.785398" velocity="1000" />
   </joint>
-  <joint name="left_wrist_pan_left_hand_joint" type="fixed">
+  <joint name="left_wrist_pan_left_wrist_pan_old_joint" type="revolute">
+    <origin rpy="-4.712389 0 0" xyz="0.002 0 0" />
+    <parent link="left_wrist_pan" />
+    <child link="left_wrist_pan_old" />
+    <axis xyz="0 0 1" />
+    <limit effort="1000" lower="-0.785398" upper="0.785398" velocity="1000" />
+  </joint>
+  <joint name="left_wrist_pan_old_left_hand_joint" type="fixed">
     <origin xyz="0.012 0 0" />
-    <parent link="left_wrist_pan" />
+    <parent link="left_wrist_pan_old" />
     <child link="left_hand" />
   </joint>
