Commit message: left wrist tilt visual added

File: nefive_description/urdf/arms.xacro (robot description, xacro)
@@ -65,5 +65,5 @@
         <cylinder length="0.034" radius="0.005" />
       </geometry>
-      <material name="green" />
+      <material name="grey" />
     </visual>
   </link>
@@ -75,6 +75,13 @@
       <material name="grey" />
     </visual>
+    <visual>
+      <origin rpy="0 1.570451 0" xyz="0.016 0 0" />
+      <geometry>
+        <cylinder length="0.032" radius="0.005" />
+      </geometry>
+      <material name="grey" />
+    </visual>
   </link>
-  <link name="left_wrist_pan_old">
+  <link name="left_wrist_tilt">
     <visual>
       <geometry>
@@ -134,14 +141,14 @@
     <limit effort="1000" lower="-0.785398" upper="0.785398" velocity="1000" />
   </joint>
-  <joint name="left_wrist_pan_left_wrist_pan_old_joint" type="revolute">
-    <origin rpy="-4.712389 0 0" xyz="0.002 0 0" />
+  <joint name="left_wrist_pan_left_wrist_tilt_joint" type="revolute">
+    <origin rpy="1.57 0 0" xyz="0.036 0 0" />
     <parent link="left_wrist_pan" />
-    <child link="left_wrist_pan_old" />
-    <axis xyz="0 0 1" />
+    <child link="left_wrist_tilt" />
+    <axis xyz="0 0 -1" />
     <limit effort="1000" lower="-0.785398" upper="0.785398" velocity="1000" />
   </joint>
-  <joint name="left_wrist_pan_old_left_hand_joint" type="fixed">
+  <joint name="left_wrist_tilt_left_hand_joint" type="fixed">
     <origin xyz="0.012 0 0" />
-    <parent link="left_wrist_pan_old" />
+    <parent link="left_wrist_tilt" />
     <child link="left_hand" />
   </joint>

Commit message: swapped out for xacro

File: nefive_description/urdf/arms.xacro (robot description, xacro)
@@ -1,8 +1,10 @@
 <?xml version="1.0"?>
 <robot xmlns:xacro="http://www.ros.org/wiki/xacro">
-  <link name="left_arm" />
-  <link name="left_shoulder_flappy">
+<link name="arms" />
+<xacro:macro name="arm" params="prefix reflect">
+  <link name="${prefix}_arm" />
+  <link name="${prefix}_shoulder_flappy">
     <visual>
-      <origin rpy="1.570451 0 0" xyz="0 0 0" />
+      <origin rpy="${pi/2} 0 0" xyz="0 0 0" />
       <geometry>
         <cylinder length="0.02" radius="0.0005" />
@@ -11,7 +13,7 @@
     </visual>
   </link>
-  <link name="left_shoulder_foreaft">
+  <link name="${prefix}_shoulder_foreaft">
     <visual>
-      <origin rpy="0 1.570451 0" xyz="0 0 0" />
+      <origin rpy="0 ${pi/2} 0" xyz="0 0 0" />
       <geometry>
         <cylinder length="0.004" radius="0.0005" />
@@ -20,5 +22,5 @@
     </visual>
   </link>
-  <link name="left_shoulder_rotate">
+  <link name="${prefix}_shoulder_rotate">
     <visual>
       <origin rpy="0 0 0" xyz="0 0 0" />
@@ -36,7 +38,7 @@
     </visual>
   </link>
-  <link name="left_elbow">
+  <link name="${prefix}_elbow">
     <visual>
-      <origin rpy="1.570451 0 0" xyz="0 0 0" />
+      <origin rpy="${pi/2} 0 0" xyz="0 0 0" />
       <geometry>
         <cylinder length="0.004" radius="0.0005" />
@@ -45,5 +47,5 @@
     </visual>
     <visual>
-      <origin rpy="0 1.570451 0" xyz="0.021 0 0" />
+      <origin rpy="0 ${pi/2} 0" xyz="0.021 0 0" />
       <geometry>
         <cylinder length="0.042" radius="0.005" />
@@ -52,7 +54,7 @@
     </visual>
   </link>
-  <link name="left_wrist_rotate">
+  <link name="${prefix}_wrist_rotate">
     <visual>
-      <origin rpy="0 1.570451 0" xyz="0 0 0" />
+      <origin rpy="0 ${pi/2} 0" xyz="0 0 0" />
       <geometry>
         <cylinder length="0.004" radius="0.0005" />
@@ -61,5 +63,5 @@
     </visual>
     <visual>
-      <origin rpy="0 1.570451 0" xyz="0.017 0 0" />
+      <origin rpy="0 ${pi/2} 0" xyz="0.017 0 0" />
       <geometry>
         <cylinder length="0.034" radius="0.005" />
@@ -68,5 +70,5 @@
     </visual>
   </link>
-  <link name="left_wrist_pan">
+  <link name="${prefix}_wrist_pan">
     <visual>
       <geometry>
@@ -76,5 +78,5 @@
     </visual>
     <visual>
-      <origin rpy="0 1.570451 0" xyz="0.016 0 0" />
+      <origin rpy="0 ${pi/2} 0" xyz="0.016 0 0" />
       <geometry>
         <cylinder length="0.032" radius="0.005" />
@@ -83,5 +85,5 @@
     </visual>
   </link>
-  <link name="left_wrist_tilt">
+  <link name="${prefix}_wrist_tilt">
     <visual>
       <geometry>
@@ -91,5 +93,5 @@
     </visual>
   </link>
-  <link name="left_hand">
+  <link name="${prefix}_hand">
     <visual>
       <geometry>
@@ -99,57 +101,65 @@
     </visual>
   </link>
-  <joint name="left_arm_left_shoulder_flappy_joint" type="revolute">
+  <joint name="arms_${prefix}_arm" type="fixed">
+    <origin rpy="0 0 0" xyz="${reflect * -0.1} 0 0" />
+    <parent link="arms" />
+    <child link="${prefix}_arm" />
+  </joint>
+  <joint name="${prefix}_arm_${prefix}_shoulder_flappy_joint" type="revolute">
     <origin rpy="0 0 0" xyz="0 0 0" />
-    <parent link="left_arm" />
-    <child link="left_shoulder_flappy" />
+    <parent link="${prefix}_arm" />
+    <child link="${prefix}_shoulder_flappy" />
+    <axis xyz="0 ${reflect * 1} 0" />
+    <limit effort="10" lower="-${pi/2}" upper="${pi/2}" velocity="1000" />
+  </joint>
+  <joint name="${prefix}_shoulder_flappy_${prefix}_shoulder_foreaft_joint" type="revolute">
+    <origin rpy="0 0 0" xyz="${reflect * -0.025} 0 0" />
+    <parent link="${prefix}_shoulder_flappy" />
+    <child link="${prefix}_shoulder_foreaft" />
+    <axis xyz="1 0 0" />
+    <limit effort="10" lower="-${pi/2}" upper="${pi/2}" velocity="1000" />
+  </joint>
+  <joint name="${prefix}_shoulder_foreaft_${prefix}_shoulder_rotate_joint" type="revolute">
+    <origin rpy="0 0 -${pi/2}" xyz="0 0 -0.067" />
+    <parent link="${prefix}_shoulder_foreaft" />
+    <child link="${prefix}_shoulder_rotate" />
+    <axis xyz="0 0 ${reflect * 1}" />
+    <limit effort="10" lower="-${pi/2}" upper="${pi/2}" velocity="1000" />
+  </joint>
+  <joint name="${prefix}_shoulder_rotate_${prefix}_elbow_joint" type="revolute">
+    <origin rpy="0 ${pi} 0" xyz="0 0 0" />
+    <parent link="${prefix}_shoulder_rotate" />
+    <child link="${prefix}_elbow" />
     <axis xyz="0 1 0" />
-    <limit effort="1000" lower="-1.570796" upper="1.570796" velocity="1000" />
+    <limit effort="10" lower="-${pi/2}" upper="${pi/2}" velocity="1000" />
   </joint>
-  <joint name="left_shoulder_flappy_left_shoulder_foreaft_joint" type="revolute">
-    <origin rpy="0 0 0" xyz="-0.025 0 0" />
-    <parent link="left_shoulder_flappy" />
-    <child link="left_shoulder_foreaft" />
+  <joint name="${prefix}_forearm_${prefix}_wrist_rotate_joint" type="revolute">
+    <origin rpy="0 0 0" xyz="0.042 0 0" />
+    <parent link="${prefix}_elbow" />
+    <child link="${prefix}_wrist_rotate" />
     <axis xyz="1 0 0" />
-    <limit effort="1000" lower="-1.570796" upper="1.570796" velocity="1000" />
+    <limit effort="10" lower="-${pi/2}" upper="${pi/2}" velocity="1000" />
   </joint>
-  <joint name="left_shoulder_foreaft_left_shoulder_rotate_joint" type="revolute">
-    <origin rpy="0 0 -1.570451" xyz="0 0 -0.067" />
-    <parent link="left_shoulder_foreaft" />
-    <child link="left_shoulder_rotate" />
+  <joint name="${prefix}_wrist_rotate_${prefix}_wrist_pan_joint" type="revolute">
+    <origin rpy="0 0 0" xyz="0.034 0 0" />
+    <parent link="${prefix}_wrist_rotate" />
+    <child link="${prefix}_wrist_pan" />
     <axis xyz="0 0 1" />
-    <limit effort="1000" lower="-1.570796" upper="1.570796" velocity="1000" />
+    <limit effort="10" lower="-${pi/2}" upper="${pi/2}" velocity="1000" />
   </joint>
-  <joint name="left_shoulder_rotate_left_elbow_joint" type="revolute">
-    <origin rpy="0 3.14 0" xyz="0 0 0" />
-    <parent link="left_shoulder_rotate" />
-    <child link="left_elbow" />
-    <axis xyz="0 1 0" />
-    <limit effort="1000" lower="-1" upper="1" velocity="1000" />
+  <joint name="${prefix}_wrist_pan_${prefix}_wrist_tilt_joint" type="revolute">
+    <origin rpy="1.57 0 0" xyz="0.036 0 0" />
+    <parent link="${prefix}_wrist_pan" />
+    <child link="${prefix}_wrist_tilt" />
+    <axis xyz="0 0 -1" />
+    <limit effort="10" lower="-${pi/2}" upper="${pi/2}" velocity="1000" />
   </joint>
-  <joint name="left_forearm_left_wrist_rotate_joint" type="revolute">
-    <origin rpy="0 0 0" xyz="0.042 0 0" />
-    <parent link="left_elbow" />
-    <child link="left_wrist_rotate" />
-    <axis xyz="1 0 0" />
-    <limit effort="1000" lower="-1.570796" upper="1.570796" velocity="1000" />
+  <joint name="${prefix}_wrist_tilt_${prefix}_hand_joint" type="fixed">
+    <origin xyz="0.012 0 0" />
+    <parent link="${prefix}_wrist_tilt" />
+    <child link="${prefix}_hand" />
   </joint>
-  <joint name="left_wrist_rotate_left_wrist_pan_joint" type="revolute">
-    <origin rpy="0 0 0" xyz="0.034 0 0" />
-    <parent link="left_wrist_rotate" />
-    <child link="left_wrist_pan" />
-    <axis xyz="0 0 1" />
-    <limit effort="1000" lower="-0.785398" upper="0.785398" velocity="1000" />
-  </joint>
-  <joint name="left_wrist_pan_left_wrist_tilt_joint" type="revolute">
-    <origin rpy="1.57 0 0" xyz="0.036 0 0" />
-    <parent link="left_wrist_pan" />
-    <child link="left_wrist_tilt" />
-    <axis xyz="0 0 -1" />
-    <limit effort="1000" lower="-0.785398" upper="0.785398" velocity="1000" />
-  </joint>
-  <joint name="left_wrist_tilt_left_hand_joint" type="fixed">
-    <origin xyz="0.012 0 0" />
-    <parent link="left_wrist_tilt" />
-    <child link="left_hand" />
-  </joint>
-  </robot>
+</xacro:macro>
+<xacro:arm prefix="left" reflect="1"/>
+<xacro:arm prefix="right" reflect="-1"/>
+</robot>

File: nefive_description/urdf/just_arms.urdf.xacro (robot description, xacro)
@@ -4,7 +4,7 @@
   <link name="shoulder_centre" />
   <joint name="shoulder_centre_left_arm_joint" type="fixed">
-    <origin xyz="-0.10 0 0" />
+    <origin xyz="0 0 0" />
     <parent link="shoulder_centre" />
-    <child link="left_arm" />
+    <child link="arms" />
   </joint>
   <link name="forward_indicator" />

Commit message: fixed the rotation issue with the full robot model

File: nefive_description/urdf/arms.xacro (robot description, xacro)
@@ -102,5 +102,5 @@
   </link>
   <joint name="arms_${prefix}_arm" type="fixed">
-    <origin rpy="0 0 0" xyz="${reflect * -0.1} 0 0" />
+    <origin rpy="0 0 0" xyz="${reflect * -0.075} 0 0" />
     <parent link="arms" />
     <child link="${prefix}_arm" />

File: nefive_description/urdf/just_arms.urdf.xacro (robot description, xacro)
@@ -3,5 +3,5 @@
   <link name="base_link" />
   <link name="shoulder_centre" />
-  <joint name="shoulder_centre_left_arm_joint" type="fixed">
+  <joint name="shoulder_centre_arms_joint" type="fixed">
     <origin xyz="0 0 0" />
     <parent link="shoulder_centre" />

File: nefive_description/urdf/torso.xacro (robot description, xacro)
@@ -29,4 +29,9 @@
   </link>
   <link name="shoulder_centre" />
+  <joint name="shoulder_centre_arms_joint" type="fixed">
+    <origin rpy="0 0 0" xyz="0 0 0" />
+    <parent link="shoulder_centre" />
+    <child link="arms" />
+  </joint>
   <joint name="base_link_lower_torso_joint" type="fixed">
     <origin rpy="0 5.497787 0" xyz="-0.0241 0 0.0285" />
@@ -45,12 +50,7 @@
   </joint>
   <joint name="chest_box_arms_joint" type="fixed">
-    <origin xyz="0.025 0 0.075" />
+    <origin rpy="0 0 -1.570451" xyz="0.025 0 0.075" />
     <parent link="chest_box" />
     <child link="shoulder_centre" />
   </joint>
-  <joint name="shoulder_centre_left_arm_joint" type="fixed">
-    <origin xyz="-0.10 0 0" />
-    <parent link="shoulder_centre" />
-    <child link="left_arm" />
-  </joint>
 </robot>

Commit message: fixed the reversed axes

File: nefive_description/urdf/arms.xacro (robot description, xacro)
@@ -110,5 +110,5 @@
     <parent link="${prefix}_arm" />
     <child link="${prefix}_shoulder_flappy" />
-    <axis xyz="0 ${reflect * 1} 0" />
+    <axis xyz="0 -1 0" />
     <limit effort="10" lower="-${pi/2}" upper="${pi/2}" velocity="1000" />
   </joint>
@@ -117,5 +117,5 @@
     <parent link="${prefix}_shoulder_flappy" />
     <child link="${prefix}_shoulder_foreaft" />
-    <axis xyz="1 0 0" />
+    <axis xyz="${reflect} 0 0" />
     <limit effort="10" lower="-${pi/2}" upper="${pi/2}" velocity="1000" />
   </joint>
@@ -124,5 +124,5 @@
     <parent link="${prefix}_shoulder_foreaft" />
     <child link="${prefix}_shoulder_rotate" />
-    <axis xyz="0 0 ${reflect * 1}" />
+    <axis xyz="0 0 -1" />
     <limit effort="10" lower="-${pi/2}" upper="${pi/2}" velocity="1000" />
   </joint>
@@ -131,5 +131,5 @@
     <parent link="${prefix}_shoulder_rotate" />
     <child link="${prefix}_elbow" />
-    <axis xyz="0 1 0" />
+    <axis xyz="0 ${reflect} 0" />
     <limit effort="10" lower="-${pi/2}" upper="${pi/2}" velocity="1000" />
   </joint>
@@ -152,5 +152,5 @@
     <parent link="${prefix}_wrist_pan" />
     <child link="${prefix}_wrist_tilt" />
-    <axis xyz="0 0 -1" />
+    <axis xyz="0 0 ${reflect}" />
     <limit effort="10" lower="-${pi/2}" upper="${pi/2}" velocity="1000" />
   </joint>

Commit message: updated moveit, added new launch file

File: nefive_description/urdf/arms.xacro (robot description, xacro)
@@ -101,4 +101,5 @@
     </visual>
   </link>
+  <link name="${prefix}_gripper" />
   <joint name="arms_${prefix}_arm" type="fixed">
     <origin rpy="0 0 0" xyz="${reflect * -0.075} 0 0" />
@@ -160,4 +161,11 @@
     <child link="${prefix}_hand" />
   </joint>
+  <joint name="${prefix}_hand_joint_${prefix}_gripper" type="revolute">
+    <origin xyz="0 0 0" />
+    <parent link="${prefix}_hand" />
+    <child link="${prefix}_gripper" />
+    <axis xyz="0 0 ${reflect}" />
+    <limit effort="10" lower="-${pi/2}" upper="${pi/2}" velocity="1000" />
+  </joint>
 </xacro:macro>
 <xacro:arm prefix="left" reflect="1"/>

File: nefive_description/urdf/head.xacro (robot description, xacro)
@@ -17,5 +17,5 @@
     </visual>
   </link>
-  <link name="head">
+  <link name="head_roll">
     <visual>
       <origin xyz="-0.0039 0 0.0283" />
@@ -26,4 +26,5 @@
     </visual>
   </link>
+  <link name="head" />
   <link name="eyes">
     <visual>
@@ -88,6 +89,13 @@
     <limit lower="-0.785398" upper="0.785398" effort="1000" velocity="1000" />
   </joint>
-  <joint name="head_tilt_head_joint" type="fixed">
+  <joint name="head_tilt_head_roll_joint" type="revolute">
+    <origin xyz="0 0 0.035" />
     <parent link="head_tilt" />
+    <child link="head_roll" />
+    <axis xyz="0 -1 0" />
+    <limit lower="-0.785398" upper="0.785398" effort="1000" velocity="1000" />
+  </joint>
+  <joint name="head_roll_head_joint" type="fixed">
+    <parent link="head_roll" />
     <child link="head" />
   </joint>
