Commit message: moving pis...

File: nefive_description/urdf/head.xacro (robot description, xacro)
@@ -73,6 +73,5 @@
     </visual>
   </link>
-  <link name="right_camera">
-  </link>
+  <link name="right_camera" />
   <joint name="chest_box_head_pan_joint" type="revolute">
     <origin xyz="0.025 0 0.0819" />
@@ -130,4 +129,5 @@
   <joint name="right_eye_inner_right_camera_joint" type="fixed">
     <parent link="right_eye_inner" />
+    <origin rpy="${-pi/2} 0 ${-pi/2}" />
     <child link="right_camera" />
   </joint>

Commit message: updated bringup and descriptions

File: nefive_description/urdf/head.xacro (robot description, xacro)
@@ -92,5 +92,5 @@
     <parent link="head_tilt" />
     <child link="head_roll" />
-    <axis xyz="0 -1 0" />
+    <axis xyz="-1 0 0" />
     <limit lower="-0.785398" upper="0.785398" effort="1000" velocity="1000" />
   </joint>
