Commit message: updated moveit config

File: nefive_moveit/config/gazebo_nefive.urdf (robot description, URDF)
Before this commit: robot nefive, 39 links, 38 joints
Joints:
- joint left_arm_left_shoulder_flappy_joint: axis 0 1 0 -> 0 -1 0
- joint left_shoulder_foreaft_left_shoulder_rotate_joint: axis 0 0 1 -> 0 0 -1
- joint left_wrist_pan_left_wrist_tilt_joint: axis 0 0 -1 -> 0 0 1
- joint right_shoulder_flappy_right_shoulder_foreaft_joint: axis 1 0 0 -> -1 0 0
- joint right_shoulder_rotate_right_elbow_joint: axis 0 1 0 -> 0 -1 0
